File: playduino_sheep_tester/digital_io_expanders.kicad_sch (KiCad schematic)
At the start: 5 parts, among them U12 ULN2003ADR, U2 MCP23017_SO, U3 MCP23017_SO

Commit message: small improvements and fixing horrible mistakes
change A3_U2 and B7_U2 because of known issues with MCP23017
https://support.microchip.com/s/article/GPA7---GPB7-Cannot-Be-Used-as-Inputs-In-MCP23017

add resistor to MCP23017 address pins

replace B3_U2 duplicate with B6_U3
Parts:
- added R111: 2k2, Resistor_SMD:R_0603_1608Metric, symbol Device:R
Connections:
- net +3V3: now also R111.1; no longer U3.15 (A0)
- net B6_U3: now reaches U3.7 (GPB6)
- new net: R111.2, U3.15 (A0)
- no-connect marks 14 -> 13
Changed lines of the file:
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@@
-	)
-	(no_connect
-		(at 237.49 85.09)
 	)
 	(no_connect
@@
 	(wire
 		(pts
+			(xy 237.49 85.09) (xy 240.03 85.09)
+		)
+		(stroke
+			(width 0)
+			(type default)
+		)
+	)
+	(wire
+		(pts
 			(xy 72.39 91.44) (xy 74.93 91.44)
 		)
@@
 	(wire
 		(pts
-			(xy 193.04 110.49) (xy 201.93 110.49)
+			(xy 182.88 110.49) (xy 187.96 110.49)
 		)
 		(stroke
@@
 	(wire
 		(pts
+			(xy 195.58 110.49) (xy 201.93 110.49)
+		)
+		(stroke
+			(width 0)
+			(type default)
+		)
+	)
+	(wire
+		(pts
 			(xy 62.23 160.02) (xy 66.04 160.02)
 		)
@@
 	(wire
 		(pts
-			(xy 193.04 107.95) (xy 193.04 110.49)
+			(xy 182.88 107.95) (xy 182.88 110.49)
 		)
 		(stroke
@@
 		(property "Intersheetrefs" "${INTERSHEET_REFS}"
 			(at 121.8209 109.22 0)
+			(effects
+				(font
+					(size 1.27 1.27)
+				)
+				(justify left)
+				(hide yes)
+			)
+		)
+	)
+	(global_label "B6_U3"
+		(shape input)
+		(at 240.03 85.09 0)
+		(fields_autoplaced yes)
+		(effects
+			(font
+				(size 1.27 1.27)
+			)
+			(justify left)
+		)
+		(property "Intersheetrefs" "${INTERSHEET_REFS}"
+			(at 249.0023 85.09 0)
 			(effects
 				(font
@@
 	(symbol
 		(lib_id "power:+3V3")
-		(at 193.04 107.95 0)
+		(at 182.88 107.95 0)
 		(unit 1)
 		(exclude_from_sim no)
@@
 		(fields_autoplaced yes)
 		(property "Reference" "#PWR010"
-			(at 193.04 111.76 0)
+			(at 182.88 111.76 0)
 			(effects
 				(font
@@
 		)
 		(property "Value" "+3V3"
-			(at 193.04 102.87 0)
+			(at 182.88 102.87 0)
 			(effects
 				(font
@@
 		)
 		(property "Footprint" ""
-			(at 193.04 107.95 0)
+			(at 182.88 107.95 0)
 			(effects
 				(font
@@
 		)
 		(property "Datasheet" ""
-			(at 193.04 107.95 0)
+			(at 182.88 107.95 0)
 			(effects
 				(font
@@
 		)
 		(property "Description" "Power symbol creates a global label with name \"+3V3\""
-			(at 193.04 107.95 0)
+			(at 182.88 107.95 0)
 			(effects
 				(font
@@
 					(unit 1)
 				)
+			)
+		)
+	)
+	(symbol
+		(lib_id "Device:R")
+		(at 191.77 110.49 90)
+		(unit 1)
+		(exclude_from_sim no)
+		(in_bom yes)
+		(on_board yes)
+		(dnp no)
+		(fields_autoplaced yes)
+		(property "Reference" "R111"
+			(at 191.77 104.14 90)
+			(effects
+				(font
+					(size 1.27 1.27)
+				)
+			)
+		)
+		(property "Value" "2k2"
+			(at 191.77 106.68 90)
+			(effects
+				(font
+					(size 1.27 1.27)
+				)
+			)
+		)
+		(property "Footprint" "Resistor_SMD:R_0603_1608Metric"
+			(at 191.77 112.268 90)
+			(effects
+				(font
+					(size 1.27 1.27)
+				)
+				(hide yes)
+			)
+		)
+		(property "Datasheet" "~"
+			(at 191.77 110.49 0)
+			(effects
+				(font
+					(size 1.27 1.27)
+				)
+				(hide yes)
+			)
+		)
+		(property "Description" "Resistor"
+			(at 191.77 110.49 0)
+			(effects
+				(font
+					(size 1.27 1.27)
+				)
+				(hide yes)
+			)
+		)
+		(pin "2"
+		)
+		(pin "1"
+		)
+		(instances
+			(project "playduino_sheep_tester"
+				(path "/88c9457a-bea2-457f-94da-c611a4bbda4a/8e4646bd-9a17-4b53-ab58-a37b75dc5ec3"
+					(reference "R111")
+					(unit 1)
+				)
