File: playduino_sheep_tester/analog inputs.kicad_sch (KiCad schematic)
At the start: 47 parts, among them U4 ADS1115IDGS, U5 ADS1115IDGS, U6 ADS1115IDGS, U7 ADS1115IDGS

Commit message: fix hex address of ADC
Other:
- note added: "ADDR: 1001010 (0x4A) READ: 10010101 WRITE: 10010100"
- note removed: "ADDR: 1001010 (0x4B) READ: 10010101 WRITE: 10010100"
Changed lines of the file:
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@@
 		)
 	)
-	(text "ADDR:  1001010 (0x4B)\nREAD:  10010101\nWRITE: 10010100"
+	(text "ADDR:  1001010 (0x4A)\nREAD:  10010101\nWRITE: 10010100"
 		(exclude_from_sim no)
 		(at 158.75 70.866 0)

Commit message: small improvements, add GPIOs to excel
Other:
- note added: "I2C / SCL (<12V)"
Changed lines of the file:
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@@
 		)
 	)
-	(text "I2C / SDA (<12V)"
+	(text "I2C / SCL (<12V)"
 		(exclude_from_sim no)
 		(at 116.586 127.254 0)
