File: playduino_sheep_tester/raspberry_pi.kicad_sch (KiCad schematic)
At the start: 37 parts, among them J4 5520259-4, J5 5520259-4, K10 G6K-2F-Y-TR DC5, K7 G6K-2F-Y-TR DC5, K8 G6K-2F-Y-TR DC5, K9 G6K-2F-Y-TR DC5, Q18 AO3416, Q19 AO3416, U1 RASPBERRY_PI_4B_4GB, U14 XL-DB3161SRBC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

Commit message: small improvements, add GPIOs to excel
Parts:
- added R112, R113: 10k, Resistor_SMD:R_0603_1608Metric, symbol Device:R
Connections:
- net GND: now also R112.2, R113.2
- net LED_BAD: now also R112.1
- net LED_GOOD: now also R113.1
